File: hardware/SimpleFlightController.kicad_sch (KiCad schematic)
At the start: 50 parts, among them J1 Screw_Terminal_01x02, J2 Screw_Terminal_01x02, U1 BMP580, U2 BQ25883RGER, U3 ICM-45686, U4 JBL-102010052, U5 LMR51430XDDCR, U6 STM32F722RET6, U7 TPS63070RNMR

Commit message: we done design
Parts:
- removed J1: Screw_Terminal_01x02, symbol Connector:Screw_Terminal_01x02
- removed U7: TPS63070RNMR, easyeda2kicad:VQFN-15_L3.0-W2.5-P0.50-BL, symbol easyeda2kicad:TPS63070RNMR
- added C19, C36: 2.2uF, Capacitor_SMD:C_0402_1005Metric, symbol Device:C
- added C20, C21, C22, C23, C24, C33: 100nF, Capacitor_SMD:C_0402_1005Metric, symbol Device:C
- added C25, C26, C27: 1uF, Capacitor_SMD:C_0402_1005Metric, symbol Device:C
- added C28: 10uF, Capacitor_SMD:C_0805_2012Metric, symbol Device:C
- added C29, C30: 20pF, Capacitor_SMD:C_0402_1005Metric, symbol Device:C
- added C31, C32: 6.8pF, Capacitor_SMD:C_0402_1005Metric, symbol Device:C
- added C34, C37: 22uF, Capacitor_SMD:C_0805_2012Metric, symbol Device:C
- added C35: 0.1uF, Capacitor_SMD:C_0402_1005Metric, symbol Device:C
- added J3, J4: Conn_01x03, Connector_PinHeader_2.54mm:PinHeader_1x03_P2.54mm_Vertical, symbol Connector_Generic:Conn_01x03
- added L3: FCM1608KF-601T03, easyeda2kicad:L0603, symbol easyeda2kicad:FCM1608KF-601T03
- added L4: 5.6uH, easyeda2kicad:IND-SMD_L3.0-W3.0, symbol Device:L
- added R20: 10K, Resistor_SMD:R_0201_0603Metric, symbol Device:R
- added R21: 100K, Resistor_SMD:R_0402_1005Metric, symbol Device:R
- added R22: 22.1K, Resistor_SMD:R_0201_0603Metric, symbol Device:R
- added SW1, SW2: TS-1088-AR02016, easyeda2kicad:SW-SMD_L3.9-W3.0-P4.45, symbol easyeda2kicad:TS-1088-AR02016
- added U8: TPS630701RNMR, easyeda2kicad:VQFN-HR-15_L3.0-W2.5-P0.50-BL_TPS63070RNMR, symbol easyeda2kicad:TPS630701RNMR
- added X1: X322525MOB4SI, easyeda2kicad:CRYSTAL-SMD_4P-L3.2-W2.5-BL, symbol easyeda2kicad:X322525MOB4SI
- added X2: Q13FC1350000400, easyeda2kicad:FC-135R_L3.2-W1.5, symbol easyeda2kicad:Q13FC1350000400
- C1, C15, C16, C17, C2: footprint (none) -> Capacitor_SMD:C_0402_1005Metric
- C10, C18: value C -> 100nF; footprint (none) -> Capacitor_SMD:C_0402_1005Metric
- C11, C12, C14: value C -> 22uF; footprint (none) -> Capacitor_SMD:C_0805_2012Metric
- C13: value C -> 10uF; footprint (none) -> Capacitor_SMD:C_0402_1005Metric
- C3, C4, C7, C8, C9: footprint (none) -> Capacitor_SMD:C_0805_2012Metric
- C5: value 44uF -> 47uF; footprint (none) -> Capacitor_SMD:C_0805_2012Metric
- C6: value C -> 10uF; footprint (none) -> Capacitor_SMD:C_0805_2012Metric
- D1: footprint (none) -> LED_SMD:LED_0402_1005Metric
- J2: footprint (none) -> TerminalBlock:TerminalBlock_Xinya_XY308-2.54-2P_1x02_P2.54mm_Horizontal
- L1: footprint Package_QFP:LQFP-48_7x7mm_P0.5mm -> easyeda2kicad:L2520
- L2: footprint Package_QFP:LQFP-48_7x7mm_P0.5mm -> easyeda2kicad:IND-SMD_L4.0-W4.0-A
- R1, R2: footprint easyeda2kicad:USB-C-SMD_TYPE-C-16PIN-2MD-073 -> Resistor_SMD:R_0201_0603Metric
- R10, R11, R12, R13, R3, R4, R5, R6, R7, R8, R9: footprint (none) -> Resistor_SMD:R_0201_0603Metric
- R14, R15, R16, R17, R18, R19: value R -> 10K; footprint (none) -> Resistor_SMD:R_0201_0603Metric
Connections:
- net BMP_SCK is gone; now on net I2C_SCL: U1.2 (SCK)
- net BMP_SDI is gone; now on net I2C_SDA: U1.4 (SDI)
- net +3V3: now also U6.1 (VBAT), U6.19 (VDD), U6.32 (VDD), U6.48 (VDD), U6.64 (VDD), C20.1, C22.1, C23.1, C24.1, C25.1, C27.1, C28.1, C34.1, C37.1, L3.1, L4.2, R21.1, SW2.1
- net +5V: now also J3.1 (Pin_1), J4.1 (Pin_1), U8.5 (FB), U8.7 (VOUT), U8.8 (VOUT)
- net BMP_INT: now also U6.56 (PB4)
- net BQ_CE: now also U6.61 (PB8)
- net BQ_INT: now also U6.57 (PB5)
- net GND: now also C6.1, C7.1, C8.1, C9.1, U2.19 (GND), U2.20 (GND), U5.1 (GND), U6.12 (VSSA), U6.18 (VSS), U6.31 (VSS), U6.47 (VSS), U6.63 (VSS), C19.2, C20.2, C21.2, C22.2, C23.2, C24.2, C25.2, C26.2, C27.2, C28.2, C29.2, C30.2, C31.2, C32.2, C33.2, C34.2, C36.2, C37.2, J3.3 (Pin_3), J4.3 (Pin_3), R20.2, R22.2, SW1.1, U8.10 (PGND), U8.15 (VSEL), U8.4 (GND), U8.6 (FB2), X1.2 (GND), X1.4 (GND)
- net I2C_SCL: now also U6.58 (PB6)
- net I2C_SDA: now also U6.59 (PB7)
- net ICM_CS: now also U6.20 (PA4)
- net ICM_INT1: now also U6.25 (PB0)
- net ICM_INT2: now also U6.26 (PB1)
- net ICM_SCK: now also U6.21 (PA5)
- net ICM_SDI: now also U6.23 (PA7)
- net ICM_SDO: now also U6.22 (PA6)
- net SD_CD: now also U6.55 (PB3)
- net SD_CLK: now also U6.53 (PC12)
- net SD_CMD: now also U6.54 (PD2)
- net SD_DAT0: now also U6.39 (PC8)
- net SD_DAT1: now also U6.40 (PC9)
- net SD_DAT2: now also U6.51 (PC10)
- net SD_DAT3: now also U6.52 (PC11)
- net USB_DN: now also U6.44 (PA11)
- net USB_DP: now also U6.45 (PA12)
- net VSYS: now also R12.1, U5.3 (VIN), U5.5 (EN), C36.1, U8.12 (VIN), U8.13 (VIN); no longer R12.2
- net at L2.1: now also U8.11 (L1)
- net at L2.2: now also U8.9 (L2)
- net VDDA: now reaches U6.13 (VDDA)
- net VDDA: now also C21.1, C26.1, L3.2
- net SERVO1: now reaches U6.14 (PA0-WKUP)
- net SERVO1: now also J3.2 (Pin_2)
- net SERVO2: now reaches U6.15 (PA1)
- net SERVO2: now also J4.2 (Pin_2)
- net LSE_IN: now reaches U6.3 (PC14-OSC32_IN)
- net LSE_IN: now also C31.1, X2.1
- net at U6.30 (VCAP_1): now also C19.1
- net LSE_OUT: now reaches U6.4 (PC15-OSC32_OUT)
- net LSE_OUT: now also C32.1, X2.2
- net HSE_IN: now reaches U6.5 (PH0-OSC_IN)
- net HSE_IN: now also C30.1, X1.1 (OSC1)
- net HSE_OUT: now reaches U6.6 (PH1-OSC_OUT)
- net HSE_OUT: now also C29.1, X1.3 (OSC2)
- net BOOT: now reaches U6.60 (BOOT0)
- net BOOT: now also R20.1, SW2.2
- net RESET: now reaches U6.7 (NRST)
- net RESET: now also C33.1, SW1.2
- net at R13.1: now also U8.2 (PG)
- net at C10.2: now also U8.3 (VAUX)
- net at U5.2 (SW): now also C35.2, L4.1
- net at U5.4 (FB): now also R21.2, R22.1
- net at U5.6 (CB): now also C35.1
- new net: R12.2, U8.1 (PS/SYNC), U8.14 (EN)
- no-connect marks 10 -> 35
Other:
- moved on the sheet: C1, C10, C11, C12, C13, C14, C15, C16, C17, C18, C2, C3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
